File: Parcial1.brd (EAGLE design)
At the start: 68.6 x 53.3 mm, 82 parts

Commit message: Versión ultimate del circuito
Parts:
- removed R10, R11, R12, R13, R14, R15, R9: 560‎Ω, AUTODESK_CIRCUITS_BREADBOARD:0207/10
- removed U2: (no value), AUTODESK_CIRCUITS_BREADBOARD:DIL16
- added U4: (no value), AUTODESK_CIRCUITS_BREADBOARD:DIL16
- moved U1 825.5 mm to (5.00, 835.6)
- moved U3 190.5 mm to (5.00, 848.3)
- moved R2 25.4 mm to (5.00, 873.7)
- moved R3 25.4 mm to (5.00, 886.4)
- moved R4 25.4 mm to (5.00, 899.1)
- moved R5 25.4 mm to (5.00, 911.8)
- moved R6 25.4 mm to (5.00, 924.5)
- moved R7 25.4 mm to (5.00, 937.2)
- moved R8 25.4 mm to (5.00, 949.9)
- moved D41 12.7 mm to (5.00, 518.1)
- moved D42 12.7 mm to (5.00, 530.8)
- moved D43 12.7 mm to (5.00, 543.5)
- moved D44 12.7 mm to (5.00, 556.2)
- moved D45 12.7 mm to (5.00, 568.9)
- moved D46 12.7 mm to (5.00, 581.6)
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Connections:
- removed net N$26 (its old number): D18.A, D21.A, D33.A, D40.A, R7.1
- removed net N$33: D2.A, D30.A, D50.A, D57.A, R15.1
- removed net N$34: D1.A, D28.A, D3.A, D49.A, R14.1
- removed net N$35: D44.A, D6.A, D7.A, D8.A, R13.1
- removed net N$36: D10.A, D11.A, D4.A, D9.A, R12.1
- removed net N$37: D12.A, D14.A, D20.A, D61.A, D62.A, R11.1
- removed net N$38: D23.A, D26.A, D38.A, D43.A, R10.1
- removed net N$39: D15.A, D16.A, D27.A, D39.A, D64.A, R9.1
- removed net N$40: D1.K, D10.K, D11.K, D12.K, D13.K, D14.K, D15.K, D16.K, D17.K, D18.K, D19.K, D2.K, D20.K, D21.K, D22.K, D23.K, D24.K, D25.K, D26.K, D27.K, D28.K, D29.K, D3.K, D30.K, D31.K, D32.K, D33.K, D34.K, D35.K, D36.K, D37.K, D38.K, D39.K, D4.K, D40.K, D41.K, D42.K, D43.K, D44.K, D45.K, D46.K, D47.K, D48.K, D49.K, D5.K, D50.K, D51.K, D52.K, D53.K, D54.K, D55.K, D56.K, D57.K, D58.K, D59.K, D6.K, D60.K, D61.K, D62.K, D63.K, D64.K, D7.K, D8.K, D9.K, U1.GND, U2.13, U2.8, U3.13, U3.7, U3.8
- new net N$22: R3.1, U3.2
- net N$1: now also D1.K, D2.K, D3.K, D4.K, D5.K, D6.K, D7.K, D8.K, R1.2; no longer R7.2, U2.1
- net N$10: now also D10.A, D18.A, D2.A, D26.A, D34.A, D42.A, D50.A, D58.A, U4.1; no longer R5.2, U2.3
- net N$11: now also D11.A, D19.A, D27.A, D3.A, D35.A, D43.A, D51.A, D59.A, U4.2; no longer U2.9
- net N$12: now also D12.A, D20.A, D28.A, D36.A, D4.A, D44.A, D52.A, D60.A, U4.3; no longer U1.9, U2.11
- net N$13: now also D13.A, D21.A, D29.A, D37.A, D45.A, D5.A, D53.A, D61.A, U4.4; no longer R14.2, U3.1
- net N$14: now also D16.A, D24.A, D32.A, D40.A, D48.A, D56.A, D64.A, D8.A, U4.7; no longer R11.2, U3.4
- net N$15: now also D15.A, D23.A, D31.A, D39.A, D47.A, D55.A, D63.A, D7.A, U4.6; no longer R9.2, U3.6
- net N$16: now also D14.A, D22.A, D30.A, D38.A, D46.A, D54.A, D6.A, D62.A, U4.5; no longer R13.2, U3.2
- net N$17: now also R2.1, U3.1; no longer U1.4, U3.12
- net N$18: now also R5.1, U3.4; no longer R10.2, U3.5
- net N$19: now also R7.1, U3.6; no longer U1.2, U3.14
- net N$2: now also D10.K, D11.K, D12.K, D13.K, D14.K, D15.K, D16.K, D9.K, R2.2; no longer R3.2, U2.4
- net N$20: now also R8.1, U3.7; no longer R15.2, U3.15
- net N$21: now also U1.GND.., U3.13, U3.8, U4.13, U4.8; no longer R12.2, U3.3
- net N$23: now also R6.1, U3.5; no longer U1.5, U3.11
- net N$24: now also R1.1, U3.15; no longer U1.5V, U2.10, U2.16, U3.10, U3.16
- net N$25: now also R4.1, U3.3; no longer D13.A, D17.A, D24.A, D41.A, D42.A, R8.1
- net N$27: now also U1.10, U4.12; no longer D22.A, D25.A, D29.A, D34.A, D63.A, R6.1
- net N$28: now also U1.11, U3.14, U4.14; no longer D5.A, D51.A, D52.A, D55.A, R5.1
- net N$29: now also U4.9; no longer D36.A, D46.A, D56.A, D60.A, R3.1
- net N$3: now also D17.K, D18.K, D19.K, D20.K, D21.K, D22.K, D23.K, D24.K, R3.2; no longer R4.2, U2.6
- net N$30: now also U1.5V, U3.10, U3.16, U4.10, U4.16; no longer D37.A, D45.A, D48.A, D53.A, R2.1
- net N$31: now also U1.9, U3.12; no longer D47.A, D54.A, D58.A, D59.A, R4.1
- net N$32: now also U1.13, U3.11, U4.11; no longer D19.A, D31.A, D32.A, D35.A, R1.1
- net N$4: now also D25.K, D26.K, D27.K, D28.K, D29.K, D30.K, D31.K, D32.K, R4.2; no longer R1.2, U2.7
- net N$5: now also D33.K, D34.K, D35.K, D36.K, D37.K, D38.K, D39.K, D40.K, R5.2; no longer R6.2, U2.2
- net N$6: now also D49.K, D50.K, D51.K, D52.K, D53.K, D54.K, D55.K, D56.K, R7.2; no longer U1.8, U2.12
- net N$7: now also D57.K, D58.K, D59.K, D60.K, D61.K, D62.K, D63.K, D64.K, R8.2; no longer R2.2, U2.5
- net N$8: now also D41.K, D42.K, D43.K, D44.K, D45.K, D46.K, D47.K, D48.K, R6.2; no longer U1.7, U2.14
- net N$9: now also D1.A, D17.A, D25.A, D33.A, D41.A, D49.A, D57.A, D9.A, U4.15; no longer R8.2, U2.15
